File: hardware/LED_8x8.sch (EAGLE design)
At the start: 3 parts

Commit message: progress, bitches
Parts:
- removed U$2: SHACKLOGO, shack:SHACKLOGO
- added IC1: 74HC595N, 74xx-eu:74HC595N
- added Q1, Q2, Q3, Q4, Q5, Q6, Q7, Q8: BC548, transistor-npn:BC548
- added R1: 2460, rcl:R-EU_R0603
- added SV1, SV2: (no value), con-lstb:MA20-1
Connections:
- new net !RST: SV1.15
- new net +3V3: SV2.1
- new net A0: SV1.16
- new net A1: SV1.17
- new net A10: SV2.4
- new net A13: SV2.3
- new net A14: SV1.3
- new net A15: SV1.4
- new net A2: SV1.18
- new net A3: SV1.19
- new net A4: SV2.19
- new net A5: SV2.18
- new net A6: SV2.17
- new net A7: SV2.16
- new net A8: SV2.6
- new net A9: SV2.5
- new net B0: SV2.15
- new net B1: SV2.14
- new net B10: SV2.12
- new net B11: SV2.11
- new net B12: SV2.10
- new net B13: SV2.9
- new net B14: SV2.8
- new net B15: SV2.7
- new net B2: SV2.13
- new net B3: SV1.5
- new net B4: SV1.6
- new net B5: SV1.7
- new net B6: SV1.8
- new net B7: SV1.9
- new net B8: SV1.10
- new net B9: SV1.11
- new net C13: SV1.12
- new net C14: SV1.13
- new net C15: SV1.14
- new net GND: IC1A.G, IC1P.GND, R1.1, SV1.2, SV2.2, U$1.GND
- new net N$1: IC1A.SER, U$1.SOUT
- new net N$2: IC1A.SCK, U$1.SCLK
- new net N$3: IC1A.RCK
- new net N$4: U$1.SIN
- new net N$5: U$1.XLAT
- new net N$6: U$1.BLANK
- new net N$7: R1.2, U$1.IREF
- new net POWERA1: Q1.E, U$3.1.A(P17)
- new net POWERA2: Q2.E, U$3.2.A(P18)
- new net POWERA3: Q3.E, U$3.3.A(P19)
- new net POWERA4: Q4.E, U$3.4.A(P20)
- new net POWERA5: Q5.E, U$3.5.A(P29)
- new net POWERA6: Q6.E, U$3.6.A(P30)
- new net POWERA7: Q7.E, U$3.7.A(P31)
- new net POWERA8: Q8.E, U$3.8.A(P32)
- new net SHIFTA1: IC1A.QA, Q1.B
- new net SHIFTA2: IC1A.QB, Q2.B
- new net SHIFTA3: IC1A.QC, Q3.B
- new net SHIFTA4: IC1A.QD, Q4.B
- new net SHIFTA5: IC1A.QE, Q5.B
- new net SHIFTA6: IC1A.QF, Q6.B
- new net SHIFTA7: IC1A.QG, Q7.B
- new net SHIFTA8: IC1A.QH, Q8.B
- new net VCC: IC1A.SCL, IC1P.VCC, Q1.C, Q2.C, Q3.C, Q4.C, Q5.C, Q6.C, Q7.C, Q8.C, U$1.VCC
- new net VUSB: SV1.1

Commit message: added schematic
Parts:
- removed SV1, SV2: (no value), con-lstb:MA20-1
- added U$2: STM32F303_BREAKOUT, shack:STM32F303_BREAKOUT
Connections:
- removed net !RST: SV1.15
- removed net +3V3: SV2.1
- removed net A0: SV1.16
- removed net A1: SV1.17
- removed net A10: SV2.4
- removed net A13: SV2.3
- removed net A14: SV1.3
- removed net A15: SV1.4
- removed net A2: SV1.18
- removed net A3: SV1.19
- removed net A4: SV2.19
- removed net A5: SV2.18
- removed net A6: SV2.17
- removed net A7: SV2.16
- removed net A8: SV2.6
- removed net A9: SV2.5
- removed net B0: SV2.15
- removed net B1: SV2.14
- removed net B10: SV2.12
- removed net B11: SV2.11
- removed net B12: SV2.10
- removed net B13: SV2.9
- removed net B14: SV2.8
- removed net B15: SV2.7
- removed net B2: SV2.13
- removed net B3: SV1.5
- removed net B4: SV1.6
- removed net B5: SV1.7
- removed net B6: SV1.8
- removed net B7: SV1.9
- removed net B8: SV1.10
- removed net B9: SV1.11
- removed net C13: SV1.12
- removed net C14: SV1.13
- removed net C15: SV1.14
- removed net N$2: IC1A.SCK, U$1.SCLK
- removed net N$3: IC1A.RCK
- removed net N$4: U$1.SIN
- removed net N$5: U$1.XLAT
- removed net N$6: U$1.BLANK
- removed net VUSB: SV1.1
- new net BLANK: U$1.BLANK, U$2.B1
- new net MOSI: U$1.SIN, U$2.A7
- new net RCK: IC1A.RCK, U$2.B2
- new net SCK: IC1A.SCK, U$1.SCLK, U$2.A5
- new net VDD: U$2.VUSB
- new net XLAT: U$1.XLAT, U$2.B0
- net GND: now also U$2.GND@1, U$2.GND@2; no longer SV1.2, SV2.2
- net VCC: now also U$2.+3V3

Commit message: schematic sucked
Connections:
- removed net VDD: U$2.VUSB
- new net +5V: Q1.C, Q2.C, Q3.C, Q4.C, Q5.C, Q6.C, Q7.C, Q8.C, U$2.VUSB
- net VCC: no longer Q1.C, Q2.C, Q3.C, Q4.C, Q5.C, Q6.C, Q7.C, Q8.C
Changed lines of the file:
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@@
 <part name="Q7" library="transistor-npn" deviceset="BC548*" device=""/>
 <part name="Q8" library="transistor-npn" deviceset="BC548*" device=""/>
-<part name="P+1" library="supply1" deviceset="VDD" device=""/>
-<part name="P+2" library="supply1" deviceset="VDD" device=""/>
-<part name="P+3" library="supply1" deviceset="VDD" device=""/>
-<part name="P+4" library="supply1" deviceset="VDD" device=""/>
-<part name="P+5" library="supply1" deviceset="VDD" device=""/>
-<part name="P+6" library="supply1" deviceset="VDD" device=""/>
-<part name="P+7" library="supply1" deviceset="VDD" device=""/>
-<part name="P+8" library="supply1" deviceset="VDD" device=""/>
 <part name="P+9" library="supply1" deviceset="VCC" device=""/>
 <part name="P+10" library="supply1" deviceset="VCC" device=""/>
@@
 <part name="GND5" library="supply1" deviceset="GND" device=""/>
 <part name="GND6" library="supply1" deviceset="GND" device=""/>
-<part name="VDD1" library="supply1" deviceset="VDD" device=""/>
+<part name="P+1" library="supply1" deviceset="+5V" device=""/>
+<part name="P+2" library="supply1" deviceset="+5V" device=""/>
+<part name="P+3" library="supply1" deviceset="+5V" device=""/>
+<part name="P+4" library="supply1" deviceset="+5V" device=""/>
+<part name="P+5" library="supply1" deviceset="+5V" device=""/>
+<part name="P+6" library="supply1" deviceset="+5V" device=""/>
+<part name="P+7" library="supply1" deviceset="+5V" device=""/>
+<part name="P+8" library="supply1" deviceset="+5V" device=""/>
+<part name="P+13" library="supply1" deviceset="+5V" device=""/>
 </parts>
 <sheets>
@@
 <instance part="Q8" gate="G$1" x="106.68" y="-43.18"/>
 <instance part="IC1" gate="P" x="38.1" y="-43.18" rot="R90"/>
-<instance part="P+1" gate="G$1" x="71.12" y="-45.72"/>
-<instance part="P+2" gate="G$1" x="71.12" y="-30.48"/>
-<instance part="P+3" gate="G$1" x="71.12" y="-15.24"/>
-<instance part="P+4" gate="G$1" x="71.12" y="0"/>
-<instance part="P+5" gate="G$1" x="114.3" y="10.16" rot="MR0"/>
-<instance part="P+6" gate="G$1" x="114.3" y="-5.08" rot="MR0"/>
-<instance part="P+7" gate="G$1" x="114.3" y="-20.32" rot="MR0"/>
-<instance part="P+8" gate="G$1" x="114.3" y="-35.56" rot="MR0"/>
 <instance part="P+9" gate="VCC" x="17.78" y="17.78"/>
 <instance part="P+10" gate="VCC" x="20.32" y="-15.24"/>
@@
 <instance part="GND5" gate="1" x="-78.74" y="93.98"/>
 <instance part="GND6" gate="1" x="-15.24" y="93.98"/>
-<instance part="VDD1" gate="G$1" x="-27.94" y="106.68"/>
+<instance part="P+1" gate="1" x="-27.94" y="106.68"/>
+<instance part="P+2" gate="1" x="71.12" y="0"/>
+<instance part="P+3" gate="1" x="114.3" y="10.16"/>
+<instance part="P+4" gate="1" x="114.3" y="-5.08"/>
+<instance part="P+5" gate="1" x="71.12" y="-15.24"/>
+<instance part="P+6" gate="1" x="71.12" y="-30.48"/>
+<instance part="P+7" gate="1" x="114.3" y="-35.56"/>
+<instance part="P+8" gate="1" x="114.3" y="-20.32"/>
+<instance part="P+13" gate="1" x="71.12" y="-45.72"/>
 </instances>
 <busses>
@@
 <net name="VCC" class="0">
 <segment>
-<pinref part="Q1" gate="G$1" pin="C"/>
-<pinref part="P+1" gate="G$1" pin="VDD"/>
-<wire x1="71.12" y1="-48.26" x2="76.2" y2="-48.26" width="0.1524" layer="91"/>
-</segment>
-<segment>
-<pinref part="Q2" gate="G$1" pin="C"/>
-<pinref part="P+2" gate="G$1" pin="VDD"/>
-<wire x1="71.12" y1="-33.02" x2="76.2" y2="-33.02" width="0.1524" layer="91"/>
-</segment>
-<segment>
-<pinref part="Q3" gate="G$1" pin="C"/>
-<pinref part="P+3" gate="G$1" pin="VDD"/>
-<wire x1="71.12" y1="-17.78" x2="76.2" y2="-17.78" width="0.1524" layer="91"/>
-</segment>
-<segment>
-<pinref part="Q4" gate="G$1" pin="C"/>
-<pinref part="P+4" gate="G$1" pin="VDD"/>
-<wire x1="71.12" y1="-2.54" x2="76.2" y2="-2.54" width="0.1524" layer="91"/>
-</segment>
-<segment>
-<pinref part="Q5" gate="G$1" pin="C"/>
-<pinref part="P+5" gate="G$1" pin="VDD"/>
-<wire x1="114.3" y1="7.62" x2="109.22" y2="7.62" width="0.1524" layer="91"/>
-</segment>
-<segment>
-<pinref part="Q6" gate="G$1" pin="C"/>
-<pinref part="P+6" gate="G$1" pin="VDD"/>
-<wire x1="114.3" y1="-7.62" x2="109.22" y2="-7.62" width="0.1524" layer="91"/>
-</segment>
-<segment>
-<pinref part="Q7" gate="G$1" pin="C"/>
-<pinref part="P+7" gate="G$1" pin="VDD"/>
-<wire x1="114.3" y1="-22.86" x2="109.22" y2="-22.86" width="0.1524" layer="91"/>
-</segment>
-<segment>
-<pinref part="Q8" gate="G$1" pin="C"/>
-<pinref part="P+8" gate="G$1" pin="VDD"/>
-<wire x1="114.3" y1="-38.1" x2="109.22" y2="-38.1" width="0.1524" layer="91"/>
-</segment>
-<segment>
 <pinref part="U$1" gate="G$1" pin="VCC"/>
 <pinref part="P+9" gate="VCC" pin="VCC"/>
@@
 <wire x1="22.86" y1="66.04" x2="17.78" y2="66.04" width="0.1524" layer="91"/>
 <wire x1="17.78" y1="66.04" x2="17.78" y2="63.5" width="0.1524" layer="91"/>
-</segment>
-</net>
-<net name="VDD" class="0">
-<segment>
-<pinref part="U$2" gate="G$1" pin="VUSB"/>
-<pinref part="VDD1" gate="G$1" pin="VDD"/>
-<wire x1="-33.02" y1="101.6" x2="-27.94" y2="101.6" width="0.1524" layer="91"/>
-<wire x1="-27.94" y1="101.6" x2="-27.94" y2="104.14" width="0.1524" layer="91"/>
 </segment>
 </net>
@@
 </segment>
 </net>
+<net name="+5V" class="0">
+<segment>
+<pinref part="U$2" gate="G$1" pin="VUSB"/>
+<wire x1="-33.02" y1="101.6" x2="-27.94" y2="101.6" width="0.1524" layer="91"/>
+<wire x1="-27.94" y1="101.6" x2="-27.94" y2="104.14" width="0.1524" layer="91"/>
+<pinref part="P+1" gate="1" pin="+5V"/>
+</segment>
+<segment>
+<pinref part="Q4" gate="G$1" pin="C"/>
+<wire x1="71.12" y1="-2.54" x2="76.2" y2="-2.54" width="0.1524" layer="91"/>
+<pinref part="P+2" gate="1" pin="+5V"/>
+</segment>
+<segment>
+<pinref part="Q5" gate="G$1" pin="C"/>
+<wire x1="114.3" y1="7.62" x2="109.22" y2="7.62" width="0.1524" layer="91"/>
+<pinref part="P+3" gate="1" pin="+5V"/>
+</segment>
+<segment>
+<pinref part="Q6" gate="G$1" pin="C"/>
+<wire x1="114.3" y1="-7.62" x2="109.22" y2="-7.62" width="0.1524" layer="91"/>
+<pinref part="P+4" gate="1" pin="+5V"/>
+</segment>
+<segment>
+<pinref part="Q3" gate="G$1" pin="C"/>
+<wire x1="71.12" y1="-17.78" x2="76.2" y2="-17.78" width="0.1524" layer="91"/>
+<pinref part="P+5" gate="1" pin="+5V"/>
+</segment>
+<segment>
+<pinref part="Q2" gate="G$1" pin="C"/>
+<wire x1="71.12" y1="-33.02" x2="76.2" y2="-33.02" width="0.1524" layer="91"/>
+<pinref part="P+6" gate="1" pin="+5V"/>
+</segment>
+<segment>
+<pinref part="Q8" gate="G$1" pin="C"/>
+<wire x1="114.3" y1="-38.1" x2="109.22" y2="-38.1" width="0.1524" layer="91"/>
+<pinref part="P+7" gate="1" pin="+5V"/>
+</segment>
+<segment>
+<pinref part="Q7" gate="G$1" pin="C"/>
+<wire x1="114.3" y1="-22.86" x2="109.22" y2="-22.86" width="0.1524" layer="91"/>
+<pinref part="P+8" gate="1" pin="+5V"/>
+</segment>
+<segment>
+<pinref part="Q1" gate="G$1" pin="C"/>
+<wire x1="71.12" y1="-48.26" x2="76.2" y2="-48.26" width="0.1524" layer="91"/>
+<pinref part="P+13" gate="1" pin="+5V"/>
+</segment>
+</net>

Commit message: finished layout
Parts:
- IC1: value 74HC595N -> 74HC595D; device 74xx-eu:74HC595N -> 74xx-eu:74HC595D
Changed lines of the file:
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@@
 <part name="U$1" library="shack" deviceset="TLC5947" device=""/>
 <part name="U$3" library="shack" deviceset="LED_RGB_8X8" device=""/>
-<part name="IC1" library="74xx-eu" deviceset="74*595" device="N" technology="HC"/>
+<part name="IC1" library="74xx-eu" deviceset="74*595" device="D" technology="HC" value="74HC595D"/>
 <part name="Q1" library="transistor-npn" deviceset="BC548*" device=""/>
 <part name="Q2" library="transistor-npn" deviceset="BC548*" device=""/>
